File: Eagle Files/QuickPSoC3V2_LongPads_04042012.brd (EAGLE design)
At the start: 67 x 60.3 mm, 26 parts, among them SW1 PSHBTTN, X1 USB-MINIB-5PIN

Commit message: Removed the 22ohm resistors on the USB lines,since it works just fine without them. Removed 10uF cap on USB +5V line. Added MiniProg3 insertion indication on silkscreen.
Edited gitignore to ignore *.s#* and *.b#* files.
Parts:
- removed C3: 10uF, SparkFun:CPOL-RADIAL-10UF-25V
- removed R1, R2: 22ohm, rcl:M0805
- moved U$2 4.93 mm to (38.7, 46.4)
Connections:
- removed net N$3: R2.1, U$1.34
- removed net N$4: R1.1, U$1.35
- net +5V: no longer C3.1
- net D+: now also U$1.35; no longer R1.2
- net D-: now also U$1.34; no longer R2.2
- net GND: no longer C3.2
Routing:
- net GND: track 89.0 -> 67.2 mm
- net D-: track 22.8 -> 32.8 mm
- net D+: track 20.5 -> 29.7 mm
- net N$4: track 8.77 -> 0.00 mm
- net N$3: track 8.64 -> 0.00 mm
Other:
- board text added: "MINIPROG3"
Changed lines of the file:
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@@
 <?xml version="1.0" encoding="utf-8"?>
 <!DOCTYPE eagle SYSTEM "eagle.dtd">
-<eagle version="6.1">
+<eagle version="6.2">
 <drawing>
 <settings>
@@
 <text x="54.2925" y="16.9545" size="1.778" layer="25" font="vector" ratio="12" rot="R180">SW1</text>
 <text x="62.23" y="6.6675" size="1.778" layer="25" rot="R90">CC-BY-SA 3.0</text>
+<wire x1="46.6725" y1="43.815" x2="58.1025" y2="43.815" width="0.4064" layer="25"/>
+<text x="59.69" y="46.0375" size="1.778" layer="25" font="vector" ratio="10" rot="R180">MINIPROG3</text>
 </plain>
 <attributes>
@@
 <element name="C5" library="rcl" package="C0805K" value="1uF" x="24.4475" y="34.29" smashed="yes" rot="R90"/>
 <element name="X1" library="SparkFun_Modified" package="USB-MINIB" value="USB-MINIB-5PIN" x="25.654" y="48.5775" smashed="yes" rot="R270"/>
-<element name="R1" library="rcl" package="M0805" value="22ohm" x="26.67" y="38.1" smashed="yes" rot="R90"/>
-<element name="R2" library="rcl" package="M0805" value="22ohm" x="28.8925" y="38.1" smashed="yes" rot="R90"/>
 <element name="RESET" library="switch-omron" package="B3F-10XX" value="PSHBTTN" x="46.355" y="28.2575" smashed="yes" rot="R180">
 <attribute name="NAME" x="42.9895" y="22.733" size="1.778" layer="25" font="vector" ratio="12"/>
@@
 <element name="H1" library="holes" package="2,8-PAD" value="MOUNT-PAD-ROUND2.8" x="3.4925" y="49.8475"/>
 <element name="H3" library="holes" package="2,8-PAD" value="MOUNT-PAD-ROUND2.8" x="55.245" y="49.8475"/>
-<element name="C3" library="SparkFun" package="CPOL-RADIAL-10UF-25V" value="10uF" x="12.3825" y="46.6725" smashed="yes" rot="R270"/>
 <element name="U$3" library="cypress" package="LOGO" value="" x="26.67" y="19.685"/>
 <element name="R3" library="rcl" package="M0805" value="1k" x="13.0175" y="18.0975" smashed="yes" rot="R180"/>
@@
 </element>
 <element name="H2" library="holes" package="2,8-PAD" value="MOUNT-PAD-ROUND2.8" x="54.9275" y="-1.27"/>
-<element name="U$2" library="SparkFun" package="OSHW-LOGO-L" value="OSHW-LOGOL" x="43.4975" y="47.625"/>
+<element name="U$2" library="SparkFun" package="OSHW-LOGO-L" value="OSHW-LOGOL" x="38.735" y="46.355"/>
 </elements>
 <signals>
@@
 <wire x1="46.99" y1="38.4175" x2="46.99" y2="41.4655" width="0.4064" layer="1"/>
 </signal>
-<signal name="N$3">
-<contactref element="U$1" pad="34"/>
-<contactref element="R2" pad="1"/>
-<wire x1="28.2575" y1="35.295" x2="28.8925" y2="37.15" width="0.3048" layer="1"/>
-<wire x1="28.2575" y1="28.6131" x2="28.2575" y2="35.295" width="0.3048" layer="1"/>
-</signal>
-<signal name="N$4">
-<contactref element="U$1" pad="35"/>
-<contactref element="R1" pad="1"/>
-<wire x1="27.6225" y1="28.6131" x2="27.6225" y2="35.295" width="0.3048" layer="1"/>
-<wire x1="27.6225" y1="35.295" x2="26.67" y2="37.15" width="0.3048" layer="1"/>
-</signal>
 <signal name="XRES">
 <contactref element="U$1" pad="27"/>
@@
 </signal>
 <signal name="D-">
-<contactref element="R2" pad="2"/>
 <contactref element="X1" pad="D+"/>
 <wire x1="25.654" y1="48.514" x2="25.654" y2="46.0775" width="0.4064" layer="1"/>
 <wire x1="26.67" y1="49.53" x2="25.654" y2="48.514" width="0.4064" layer="1"/>
-<wire x1="28.8925" y1="39.05" x2="28.8925" y2="40.3225" width="0.4064" layer="1"/>
-<wire x1="28.8925" y1="40.3225" x2="29.5275" y2="41.91" width="0.4064" layer="1"/>
-<wire x1="29.5275" y1="41.91" x2="31.115" y2="41.91" width="0.4064" layer="1"/>
-<wire x1="31.115" y1="41.91" x2="33.3375" y2="44.45" width="0.4064" layer="1"/>
-<wire x1="33.3375" y1="44.45" x2="33.3375" y2="48.26" width="0.4064" layer="1"/>
 <wire x1="33.3375" y1="48.26" x2="32.0675" y2="49.53" width="0.4064" layer="1"/>
 <wire x1="32.0675" y1="49.53" x2="26.67" y2="49.53" width="0.4064" layer="1"/>
+<contactref element="U$1" pad="34"/>
+<wire x1="28.2575" y1="28.6131" x2="28.2575" y2="39.6875" width="0.3048" layer="1"/>
+<wire x1="28.2575" y1="39.6875" x2="33.3375" y2="44.7675" width="0.3048" layer="1"/>
+<wire x1="33.3375" y1="44.7675" x2="33.3375" y2="48.26" width="0.4064" layer="1"/>
 </signal>
 <signal name="D+">
-<contactref element="R1" pad="2"/>
 <contactref element="X1" pad="D-"/>
-<wire x1="26.67" y1="39.05" x2="26.67" y2="39.37" width="0.3048" layer="1"/>
-<wire x1="26.67" y1="39.37" x2="26.67" y2="40.3225" width="0.4064" layer="1"/>
-<wire x1="26.67" y1="40.3225" x2="29.21" y2="42.8625" width="0.4064" layer="1"/>
-<wire x1="29.21" y1="42.8625" x2="30.7975" y2="42.8625" width="0.4064" layer="1"/>
-<wire x1="30.7975" y1="42.8625" x2="32.385" y2="44.7675" width="0.4064" layer="1"/>
-<wire x1="32.385" y1="44.7675" x2="32.385" y2="47.9425" width="0.4064" layer="1"/>
 <wire x1="32.385" y1="47.9425" x2="31.75" y2="48.5775" width="0.4064" layer="1"/>
 <wire x1="26.454" y1="48.044" x2="26.454" y2="46.0775" width="0.4064" layer="1"/>
 <wire x1="26.9875" y1="48.5775" x2="26.454" y2="48.044" width="0.4064" layer="1"/>
 <wire x1="31.75" y1="48.5775" x2="26.9875" y2="48.5775" width="0.4064" layer="1"/>
+<contactref element="U$1" pad="35"/>
+<wire x1="27.6225" y1="28.6131" x2="27.6225" y2="40.005" width="0.3048" layer="1"/>
+<wire x1="32.385" y1="47.9425" x2="32.385" y2="44.7675" width="0.4064" layer="1"/>
+<wire x1="32.385" y1="44.7675" x2="27.6225" y2="40.005" width="0.3048" layer="1"/>
 </signal>
 <signal name="GND">
 <contactref element="X1" pad="GND"/>
-<contactref element="C3" pad="2"/>
 <contactref element="JP4" pad="18"/>
 <contactref element="JP4" pad="20"/>
@@
 <wire x1="44.45" y1="3.048" x2="46.99" y2="3.048" width="0.3048" layer="1"/>
 <wire x1="46.99" y1="3.048" x2="49.53" y2="3.048" width="0.3048" layer="1"/>
-<wire x1="2.2225" y1="48.26" x2="12.3825" y2="47.9425" width="0.3048" layer="1"/>
 <wire x1="11.7475" y1="25.0825" x2="12.065" y2="25.03" width="0.3048" layer="1"/>
 <wire x1="12.065" y1="25.03" x2="15.5575" y2="24.8125" width="0.3048" layer="1"/>
 <wire x1="7.62" y1="24.495" x2="7.62" y2="27.305" width="0.3048" layer="1"/>
 <wire x1="24.054" y1="47.9425" x2="24.054" y2="46.0775" width="0.4064" layer="1"/>
-<wire x1="12.3825" y1="47.9425" x2="24.054" y2="47.9425" width="0.4064" layer="1"/>
 <wire x1="26.3525" y1="28.6131" x2="26.3525" y2="34.925" width="0.3048" layer="1"/>
 <wire x1="26.3525" y1="34.925" x2="24.4475" y2="35.29" width="0.3048" layer="1"/>
@@
 <contactref element="JP4" pad="1"/>
 <contactref element="X1" pad="VBUS"/>
-<contactref element="C3" pad="1"/>
 <wire x1="1.27" y1="3.048" x2="1.27" y2="15.24" width="1.778" layer="1"/>
 <wire x1="17.78" y1="40.9575" x2="22.86" y2="40.9575" width="0.4064" layer="16"/>
-<wire x1="4.7625" y1="45.4025" x2="12.3825" y2="45.4025" width="1.778" layer="1"/>
 <wire x1="1.27" y1="41.91" x2="4.7625" y2="45.4025" width="1.778" layer="1"/>
 <wire x1="1.27" y1="15.24" x2="1.27" y2="41.91" width="1.778" layer="1"/>
-<wire x1="12.3825" y1="45.4025" x2="16.51" y2="45.4025" width="1.778" layer="1"/>
 <wire x1="16.51" y1="45.4025" x2="17.78" y2="44.45" width="1.778" layer="1"/>
 <wire x1="17.78" y1="44.45" x2="17.78" y2="40.9575" width="1.778" layer="1"/>
@@
 <via x="22.86" y="40.9575" extent="1-16" drill="1" diameter="1.016" shape="square" alwaysstop="yes"/>
 <via x="17.78" y="40.9575" extent="1-16" drill="1" diameter="1.016" shape="square" alwaysstop="yes"/>
+<wire x1="4.7625" y1="45.4025" x2="16.51" y2="45.4025" width="1.778" layer="1"/>
 </signal>
 <signal name="N$1">
